File: R.A.W.R/MCU.kicad_sch (KiCad schematic)
At the start: 27 parts, among them J2 SM03B-SRSS-TB(LF)(SN), SW1 434133025816, SW2 434133025816, U3 RP2354A, Y3 ABM8-272-T3

Commit message: Added some footprints and USB-C receptacle
Parts:
- added J4: USB_C_Receptacle_USB2.0_14P, Connector_USB:USB_C_Receptacle_Amphenol_12401610E4-2A, symbol Connector:USB_C_Receptacle_USB2.0_14P
- added R32, R33: 5.1k, Resistor_SMD:R_0805_2012Metric_Pad1.20x1.40mm_HandSolder, symbol Device:R
- C32, C33, C34: footprint (none) -> Capacitor_SMD:C_0402_1005Metric_Pad0.74x0.62mm_HandSolder; Field5 (none) -> M1005; Field6 (none) -> 6.3V; Field7 (none) -> X5R; Field8 (none) -> 20%
- C35, C36, C37, C38, C39, C40, C41, C42, C43, C44, C45, C46: footprint (none) -> Capacitor_SMD:C_0402_1005Metric_Pad0.74x0.62mm_HandSolder
- J2: footprint Package_DFN_QFN:NXP_LQFN-48-1EP_7x7mm_P0.5mm_EP3.5x3.5mm_16xMask0.45x0.45_ThermalVias -> (none)
- L4: footprint Package_SO:SOIC-20W_7.5x12.8mm_P1.27mm -> RAWR:AOTAB201610S3R3101T; Field5 (none) -> 2.1A
- R21: footprint QFN40P1000X1000X90-81N-D -> Resistor_SMD:R_0402_1005Metric_Pad0.72x0.64mm_HandSolder; Field5 (none) -> 1%; Field6 (none) -> 63mW; Field7 (none) -> M1005
- R22, R23, R24, R25, R26: footprint QFN40P1000X1000X90-81N-D -> Resistor_SMD:R_0402_1005Metric_Pad0.72x0.64mm_HandSolder
- SW1, SW2: footprint Button_Switch_SMD:Nidec_Copal_CAS-120A -> (none)
- U3: footprint Package_DFN_QFN:QFN-60-1EP_7x7mm_P0.4mm_EP3.4x3.4mm -> Package_DFN_QFN:QFN-60-1EP_7x7mm_P0.4mm_EP3.4x3.4mm_ThermalVias
- Y3: footprint (none) -> RAWR:ABM8272T3
Connections:
- net GND: now also J4.A1 (GND), J4.A12 (GND), J4.B1 (GND), J4.B12 (GND), J4.SH (SHIELD), R32.2, R33.2
- net USB_DM: now also J4.A7 (D-), J4.B7 (D-)
- net USB_DP: now also J4.A6 (D+), J4.B6 (D+)
- new net: J4.B5 (CC2), R33.1
- new net: J4.A4 (VBUS), J4.A9 (VBUS), J4.B4 (VBUS), J4.B9 (VBUS)
- new net: J4.A5 (CC1), R32.1
- no-connect marks 5 -> 6

Commit message: Finished assignment of footprints
Parts:
- J2: footprint (none) -> RAWR:SM03BSRSSTBLFSN
- SW1, SW2: footprint (none) -> RAWR:434133025816
Changed lines of the file:
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@@
 			)
 		)
-		(property "Footprint" ""
+		(property "Footprint" "RAWR:SM03BSRSSTBLFSN"
 			(at 100.33 166.37 0)
 			(hide yes)
@@
 			)
 		)
-		(property "Footprint" ""
+		(property "Footprint" "RAWR:434133025816"
 			(at 81.28 92.71 0)
 			(hide yes)
@@
 			)
 		)
-		(property "Footprint" ""
+		(property "Footprint" "RAWR:434133025816"
 			(at 83.82 110.49 0)
 			(hide yes)

Commit message: Added charger, 3v3 regulator and 10v5 stepup
Parts:
- U3: footprint Package_DFN_QFN:QFN-60-1EP_7x7mm_P0.4mm_EP3.4x3.4mm_ThermalVias -> Package_DFN_QFN:QFN-60-1EP_7x7mm_P0.4mm_EP3.4x3.4mm
Connections:
- net +1V1: no longer U3.23 (DVDD), U3.39 (DVDD), U3.50 (VREG_FB), U3.6 (DVDD)
- net +3V3: no longer U3.53 (USB_OTP_VDD), U3.54 (QSPI_IOVDD)
- net GND: no longer U3.47 (VREG_PGND)
- net VREG_LX: now also U3.53 (USB_OTP_VDD); no longer U3.48 (VREG_LX)
- net VBUS: now reaches J4.A4 (VBUS), J4.A9 (VBUS), J4.B4 (VBUS), J4.B9 (VBUS)
- new net: U3.23 (DVDD), U3.39 (DVDD), U3.6 (DVDD)
- no-connect marks 6 -> 5
Changed lines of the file:
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@@
 	)
 	(junction
+		(at 232.41 105.41)
+		(diameter 0)
+		(color 0 0 0 0)
+	)
+	(junction
 		(at 91.44 166.37)
 		(diameter 0)
@@
 	)
 	(no_connect
-		(at 229.87 106.68)
-	)
-	(no_connect
 		(at 104.14 128.27)
 	)
@@
 	(wire
 		(pts
+			(xy 229.87 106.68) (xy 232.41 106.68)
+		)
+		(stroke
+			(width 0)
+			(type default)
+		)
+	)
+	(wire
+		(pts
 			(xy 233.68 119.38) (xy 229.87 119.38)
 		)
@@
 	(wire
 		(pts
+			(xy 232.41 106.68) (xy 232.41 105.41)
+		)
+		(stroke
+			(width 0)
+			(type default)
+		)
+	)
+	(wire
+		(pts
 			(xy 140.97 74.93) (xy 140.97 38.1)
 		)
@@
 			)
 		)
-		(property "Description" "10%"
+		(property "Description" "Unpolarized capacitor"
 			(at 181.61 43.942 0)
 			(show_name no)
@@
 			)
 		)
-		(property "Description" "10%"
+		(property "Description" "Unpolarized capacitor"
 			(at 223.52 68.072 0)
 			(show_name no)
@@
 			)
 		)
-		(property "Description" "10%"
+		(property "Description" "Unpolarized capacitor"
 			(at 171.45 43.942 0)
 			(show_name no)
@@
 			)
 		)
-		(property "Description" "10%"
+		(property "Description" "Unpolarized capacitor"
 			(at 181.61 68.072 0)
 			(show_name no)
@@
 	)
 	(symbol
+		(lib_id "power:VBUS")
+		(at 232.41 105.41 0)
+		(unit 1)
+		(body_style 1)
+		(exclude_from_sim no)
+		(in_bom yes)
+		(on_board yes)
+		(in_pos_files yes)
+		(dnp no)
+		(fields_autoplaced yes)
+		(property "Reference" "#PWR061"
+			(at 232.41 109.22 0)
+			(hide yes)
+			(show_name no)
+			(do_not_autoplace no)
+			(effects
+				(font
+					(size 1.27 1.27)
+				)
+			)
+		)
+		(property "Value" "VBUS"
+			(at 232.41 100.33 0)
+			(show_name no)
+			(do_not_autoplace no)
+			(effects
+				(font
+					(size 1.27 1.27)
+				)
+			)
+		)
+		(property "Footprint" ""
+			(at 232.41 105.41 0)
+			(hide yes)
+			(show_name no)
+			(do_not_autoplace no)
+			(effects
+				(font
+					(size 1.27 1.27)
+				)
+			)
+		)
+		(property "Datasheet" ""
+			(at 232.41 105.41 0)
+			(hide yes)
+			(show_name no)
+			(do_not_autoplace no)
+			(effects
+				(font
+					(size 1.27 1.27)
+				)
+			)
+		)
+		(property "Description" "Power symbol creates a global label with name \"VBUS\""
+			(at 232.41 105.41 0)
+			(hide yes)
+			(show_name no)
+			(do_not_autoplace no)
+			(effects
+				(font
+					(size 1.27 1.27)
+				)
+			)
+		)
+		(pin "1"
+		)
+		(instances
+			(project "R.A.W.R"
+				(path "/2e25a181-2d09-4815-b900-9881fc510404/d7847df5-016b-4dd9-9995-9480afcd9cf7"
+					(reference "#PWR061")
+					(unit 1)
+				)
+			)
+		)
+	)
+	(symbol
 		(lib_id "Device:C")
 		(at 97.79 64.77 0)
@@
 	)
 	(symbol
+		(lib_id "power:PWR_FLAG")
+		(at 232.41 105.41 270)
+		(unit 1)
+		(body_style 1)
+		(exclude_from_sim no)
+		(in_bom yes)
+		(on_board yes)
+		(in_pos_files yes)
+		(dnp no)
+		(fields_autoplaced yes)
+		(property "Reference" "#FLG02"
+			(at 234.315 105.41 0)
+			(hide yes)
+			(show_name no)
+			(do_not_autoplace no)
+			(effects
+				(font
+					(size 1.27 1.27)
+				)
+			)
+		)
+		(property "Value" "PWR_FLAG"
+			(at 236.22 105.4099 90)
+			(show_name no)
+			(do_not_autoplace no)
+			(effects
+				(font
+					(size 1.27 1.27)
+				)
+				(justify left)
+			)
+		)
+		(property "Footprint" ""
+			(at 232.41 105.41 0)
+			(hide yes)
+			(show_name no)
+			(do_not_autoplace no)
+			(effects
+				(font
+					(size 1.27 1.27)
+				)
+			)
+		)
+		(property "Datasheet" ""
+			(at 232.41 105.41 0)
+			(hide yes)
+			(show_name no)
+			(do_not_autoplace no)
+			(effects
+				(font
+					(size 1.27 1.27)
+				)
+			)
+		)
+		(property "Description" "Special symbol for telling ERC where power comes from"
+			(at 232.41 105.41 0)
+			(hide yes)
+			(show_name no)
+			(do_not_autoplace no)
+			(effects
+				(font
+					(size 1.27 1.27)
+				)
+			)
+		)
+		(pin "1"
+		)
+		(instances
+			(project "R.A.W.R"
+				(path "/2e25a181-2d09-4815-b900-9881fc510404/d7847df5-016b-4dd9-9995-9480afcd9cf7"
+					(reference "#FLG02")
+					(unit 1)
+				)
+			)
+		)
+	)
+	(symbol
 		(lib_id "Device:C")
 		(at 88.9 78.74 0)
@@
 			)
 		)
-		(property "Description" "10%"
+		(property "Description" "Unpolarized capacitor"
 			(at 191.77 43.942 0)
 			(show_name no)
@@
 			)
 		)
-		(property "Description" "10%"
+		(property "Description" "Unpolarized capacitor"
 			(at 171.45 68.072 0)
 			(show_name no)
@@
 			)
 		)
-		(property "Description" "5%"
+		(property "Description" "Unpolarized capacitor"
 			(at 75.438 151.13 0)
 			(show_name no)
@@
 			)
 		)
-		(property "Description" "10%"
+		(property "Description" "Unpolarized capacitor"
 			(at 212.09 68.072 0)
 			(show_name no)
@@
 			)
 		)
-		(property "Footprint" "Package_DFN_QFN:QFN-60-1EP_7x7mm_P0.4mm_EP3.4x3.4mm_ThermalVias"
+		(property "Footprint" "Package_DFN_QFN:QFN-60-1EP_7x7mm_P0.4mm_EP3.4x3.4mm"
 			(at 129.54 120.65 0)
 			(hide yes)
@@
 			)
 		)
-		(property "Description" "5%"
+		(property "Description" "Unpolarized capacitor"
 			(at 74.422 130.81 0)
 			(show_name no)
@@
 			)
 		)
-		(property "Description" "10%"
+		(property "Description" "Unpolarized capacitor"
 			(at 201.93 68.072 0)
 			(show_name no)
@@
 			)
 		)
-		(property "Description" "10%"
+		(property "Description" "Unpolarized capacitor"
 			(at 191.77 68.072 0)
 			(show_name no)
@@
 			)
 		)
-		(property "Description" "10%"
+		(property "Description" "Unpolarized capacitor"
 			(at 234.95 68.072 0)
 			(show_name no)

Commit message: Finished adding footprints
Parts:
- removed C35, C36, C37, C38, C39, C40, C41: 100n, Capacitor_SMD:C_0402_1005Metric_Pad0.74x0.62mm_HandSolder, symbol Device:C
- added C74, C75, C76, C77, C78, C79, C80: 100n, Capacitor_SMD:C_0402_1005Metric_Pad0.74x0.62mm_HandSolder, symbol Device:C
- C42, C43, C44: Field8 (none) -> 10%
- C45, C46: Field8 (none) -> 5%
Connections:
- net +1V1: now also U3.23 (DVDD), U3.39 (DVDD), U3.50 (VREG_FB), U3.6 (DVDD), C79.1, C80.1; no longer C43.1, C44.1
- net +3V3: now also C43.1, C44.1, U3.53 (USB_OTP_VDD), U3.54 (QSPI_IOVDD), C74.1, C75.1, C76.1, C77.1, C78.1
- net GND: now also U3.47 (VREG_PGND), C74.2, C75.2, C76.2, C77.2, C78.2, C79.2, C80.2
- net VREG_LX: now also U3.48 (VREG_LX); no longer U3.53 (USB_OTP_VDD)
